File: CADs/HeatControl/HeatControl.kicad_pcb (KiCad board)
At the start: 2 copper layers, 16 parts, among them J1 240VRelais, J2 24VPins, J3 Temp_Sensor, J4 TempSensor, J6 Fan, K1 TIANBO-HJR-4102-L, Q1 2N2219

Commit message: Update board
Parts:
- removed J1: 240VRelais, Connector_PinHeader_2.54mm:PinHeader_1x03_P2.54mm_Vertical
- added 240V: 240VRelais, Connector_PinHeader_2.54mm:PinHeader_1x03_P2.54mm_Vertical, F.Cu at (252.5, 16.8)
- added C2: 100µF, Capacitor_THT:CP_Radial_D8.0mm_P3.80mm, F.Cu at (263.4, 57.1)
- added G***: LOGO, Customs:bees, F.Cu at (260.4, 25.7)
- added G***: LOGO, Customs:openHardware, F.Cu at (260.1, 45.7)
- 10µF: renamed from C1; value CP1 -> 10µF
- Q1: footprint Package_TO_SOT_THT:TO-92 -> Package_TO_SOT_THT:TO-92_Inline
- R1: value R -> 1K
- R2: value R -> 4.7K
- R3: value R -> 3M; footprint Resistor_SMD:R_0805_2012Metric_Pad1.15x1.40mm_HandSolder -> Resistor_THT:R_Axial_DIN0207_L6.3mm_D2.5mm_P2.54mm_Vertical
- R4: value R -> 470
- R5: value R -> 4,7K
- moved R1 6.59 mm to (272.5, 18.5)
- moved D1 5.79 mm to (272.7, 52.8)
- moved R2 5.62 mm to (256.8, 53.8), turned to 90 degrees
- moved R3 5.59 mm to (261.1, 20.1)
- moved 10µF 4.66 mm to (256.5, 18.9)
- moved Raspi 3.50 mm to (282.4, 21.1)
- moved D2 3.34 mm to (258.1, 38.2)
- moved 24V 2.59 mm to (252.5, 28.2)
- moved Fan 2.59 mm to (252.5, 36.1)
- moved Temp1 2.59 mm to (252.5, 43.9)
- moved Temp2 2.59 mm to (252.5, 54.1)
- moved K1 2.34 mm to (273.1, 47.8)
- moved Q1 1.55 mm to (268.0, 25.4)
- moved R4 1.55 mm to (274.1, 29.7)
- moved R5 1.55 mm to (274.1, 23.1)
- renumbered J2 to 24V, J6 to Fan, J3 to Temp1, J4 to Temp2
Routing:
- net +5V: track 0.00 -> 166.3 mm
- net /TempData: track 0.00 -> 61.2 mm, vias 0 -> 1
- net Net-(D2-Pad2): track 0.00 -> 26.9 mm
- net /24VGND: track 0.00 -> 26.5 mm, vias 0 -> 4
- net Net-(C1-Pad1): track 0.00 -> 19.8 mm
- net +24V: track 0.00 -> 18.5 mm
- net /HeaterSignal: track 0.00 -> 15.3 mm, vias 0 -> 1
- net Net-(K1-Pad8): track 0.00 -> 11.7 mm
- net Net-(Q1-Pad2): track 0.00 -> 11.5 mm
- net /FanSignal: track 0.00 -> 6.68 mm, vias 0 -> 1
- net GND: vias 0 -> 16
- added copper zone on B.Cu, net GND
- added copper zone on F.Cu, net GND
Other:
- board text added: "+24V"
- board text added: "+5V"
- board text added: "Data"

Commit message: Board rework
Parts:
- removed 10µF: 10µF, Capacitor_Tantalum_SMD:CP_EIA-3216-18_Kemet-A_Pad1.58x1.35mm_HandSolder
- removed 240V: 240VRelais, Connector_PinHeader_2.54mm:PinHeader_1x03_P2.54mm_Vertical
- removed the G*** at (260.1, 45.7)
- removed Raspi: RaspPi, Customs:PinHeader_2x13_P2.54mm_Vertical_Mirrored
- added ?: RaspPi, Customs:PinHeader_2x13_P2.54mm_Vertical_Mirrored, B.Cu at (280.7, 21.6)
- added G***: LOGO, Customs:openHardwareSmall, F.Cu at (256.3, 17.3)
- added Heater: 240VRelais, Connector_PinHeader_2.54mm:PinHeader_1x03_P2.54mm_Vertical, F.Cu at (251.0, 37.8)
- added Q2: 2N2219, Package_TO_SOT_THT:TO-92_Inline, F.Cu at (258.8, 40.1)
- C2: footprint Capacitor_THT:CP_Radial_D8.0mm_P3.80mm -> Capacitor_THT:CP_Radial_D8.0mm_P3.50mm
- R1: value 1K -> 470
- R3: value 3M -> 4.7K; footprint Resistor_THT:R_Axial_DIN0207_L6.3mm_D2.5mm_P2.54mm_Vertical -> Resistor_SMD:R_0805_2012Metric_Pad1.15x1.40mm_HandSolder
- moved R2 37.2 mm to (274.3, 21.1)
- moved C2 30.0 mm to (261.9, 27.2), turned to 0 degrees
- moved 24V 29.0 mm to (251.0, 57.1)
- moved Temp2 27.0 mm to (251.0, 27.2)
- moved Temp1 26.7 mm to (251.0, 17.3)
- moved R1 20.7 mm to (261.1, 35.8)
- moved Fan 16.3 mm to (251.0, 52.3), turned to 180 degrees
- moved R3 15.2 mm to (257.6, 34.8), turned to 270 degrees
- moved Q1 14.7 mm to (268.5, 40.1), turned to 180 degrees
- moved R5 13.6 mm to (267.2, 34.8)
- moved D2 12.8 mm to (256.8, 50.9), turned to 270 degrees
- moved K1 11.0 mm to (270.5, 58.4)
- moved G*** 9.34 mm to (267.0, 19.1)
- moved R4 6.92 mm to (270.8, 35.8), turned to 0 degrees
- moved D1 5.75 mm to (277.6, 55.8), turned to 90 degrees
Connections:
- R2 pad 1: +5V -> /TempData
- R2 pad 2: /TempData -> +3V3
- Temp1 pad 1: GND -> +5V
- Temp1 pad 3: +5V -> GND
- Temp2 pad 1: GND -> +5V
- Temp2 pad 3: +5V -> GND
Routing:
- net +5V: track 166.3 -> 130.0 mm
- net /24VGND: track 26.5 -> 12.5 mm, vias 4 -> 0
- net Net-(Q2-Pad2): track 19.8 -> 6.85 mm
- net /TempData: track 61.2 -> 50.4 mm, vias 1 -> 4
- net Net-(240VRelay1-Pad1): track 0.00 -> 6.73 mm
- net +24V: track 18.5 -> 12.2 mm
- net +3V3: track 0.00 -> 5.76 mm
- net Net-(Q1-Pad2): track 11.5 -> 6.85 mm
- net /HeaterSignal: track 15.3 -> 19.9 mm
- net /FanSignal: track 6.68 -> 9.12 mm
- net Net-(K1-Pad8): track 11.7 -> 12.6 mm
- net GND: vias 16 -> 6
Other:
- board text added: "Heater.Pi"
- board text added: "Sig"
- board text removed: "Data"
- board text removed: "Heater.Pi 2"
