File: CADs/HeatControl/HeatControl.kicad_pcb (KiCad board)
At the start: 2 copper layers, 19 parts, among them K1 TIANBO-HJR-4102-L, Q1 2N2219, Q2 2N2219

Commit message: Add board outline
Other:
- board outline added: 35.3 x 49.3 mm
Changed lines of the file:
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@@
   (general
     (thickness 1.6)
-    (drawings 11)
+    (drawings 15)
     (tracks 101)
     (zones 0)
@@
       (outputformat 1)
       (mirror false)
-      (drillshape 1)
+      (drillshape 0)
       (scaleselection 1)
-      (outputdirectory ""))
+      (outputdirectory "../../../../../Desktop/Gerber/HeatControl/"))
   )
   (net 0 "")
@@
       (xy -1.650999 0.082931) (xy -1.650999 -1.650999) (xy 1.651 -1.650999) (xy 1.651 1.651)) (layer F.SilkS) (width 0.01))
   )
+  (gr_line (start 247.904 62.992) (end 247.904 13.716) (layer Edge.Cuts) (width 0.1))
+  (gr_line (start 283.21 62.992) (end 247.904 62.992) (layer Edge.Cuts) (width 0.1))
+  (gr_line (start 283.21 13.716) (end 283.21 62.992) (layer Edge.Cuts) (width 0.1))
+  (gr_line (start 247.904 13.716) (end 283.21 13.716) (layer Edge.Cuts) (width 0.1))
   (gr_text +5V (at 281.686 15.748) (layer F.SilkS)
     (effects (font (size 0.4 0.4) (thickness 0.1)))
