File: CADs/HeatControl/HeatControl.sch (KiCad schematic (older format))
At the start: 16 parts, among them J1 240VRelais, J2 24VPins, J3 Temp_Sensor, J4 TempSensor, J5 RaspPi, J6 Fan, K1 TIANBO-HJR-4102-L, Q1 2N2219

Commit message: Update board
Parts:
- added C2: 100µF, Capacitor_THT:CP_Radial_D8.0mm_P3.80mm, symbol Device:CP1
- C1: value CP1 -> 10µF
- Q1: footprint Package_TO_SOT_THT:TO-92 -> Package_TO_SOT_THT:TO-92_Inline
- R1: value R -> 1K
- R2: value R -> 4.7K
- R3: value R -> 3M; footprint Resistor_SMD:R_0805_2012Metric_Pad1.15x1.40mm_HandSolder -> Resistor_THT:R_Axial_DIN0207_L6.3mm_D2.5mm_P2.54mm_Vertical
- R4: value R -> 470
- R5: value R -> 4,7K
Connections:
- net +5V: now also C2.1
- net GND: now also C2.2
Changed lines of the file:
@@
 F 0 "Q1" H 9191 4046 50  0000 L CNN
 F 1 "2N2219" H 9191 3955 50  0000 L CNN
-F 2 "Package_TO_SOT_THT:TO-92" H 9200 3925 50  0001 L CIN
+F 2 "Package_TO_SOT_THT:TO-92_Inline" H 9200 3925 50  0001 L CIN
 F 3 "http://www.onsemi.com/pub_link/Collateral/2N2219-D.PDF" H 9000 4000 50  0001 L CNN
 	1    9000 4000
@@
 P 8500 4000
 F 0 "R4" V 8293 4000 50  0000 C CNN
-F 1 "R" V 8384 4000 50  0000 C CNN
+F 1 "470" V 8384 4000 50  0000 C CNN
 F 2 "Resistor_SMD:R_0805_2012Metric_Pad1.15x1.40mm_HandSolder" V 8430 4000 50  0001 C CNN
 F 3 "~" H 8500 4000 50  0001 C CNN
@@
 P 8700 4300
 F 0 "R5" H 8630 4254 50  0000 R CNN
-F 1 "R" H 8630 4345 50  0000 R CNN
+F 1 "4,7K" H 8630 4345 50  0000 R CNN
 F 2 "Resistor_SMD:R_0805_2012Metric_Pad1.15x1.40mm_HandSolder" V 8630 4300 50  0001 C CNN
 F 3 "~" H 8700 4300 50  0001 C CNN
@@
 P 3450 5500
 F 0 "R2" V 3243 5500 50  0000 C CNN
-F 1 "R" V 3334 5500 50  0000 C CNN
+F 1 "4.7K" V 3334 5500 50  0000 C CNN
 F 2 "Resistor_SMD:R_0805_2012Metric_Pad1.15x1.40mm_HandSolder" V 3380 5500 50  0001 C CNN
 F 3 "~" H 3450 5500 50  0001 C CNN
@@
 L power:GND #PWR0112
 U 1 1 5FE32A0A
-P 2150 5850
-F 0 "#PWR0112" H 2150 5600 50  0001 C CNN
-F 1 "GND" H 2155 5677 50  0000 C CNN
-F 2 "" H 2150 5850 50  0001 C CNN
-F 3 "" H 2150 5850 50  0001 C CNN
-	1    2150 5850
+P 2150 5600
+F 0 "#PWR0112" H 2150 5350 50  0001 C CNN
+F 1 "GND" H 2155 5427 50  0000 C CNN
+F 2 "" H 2150 5600 50  0001 C CNN
+F 3 "" H 2150 5600 50  0001 C CNN
+	1    2150 5600
 	-1   0    0    1
 $EndComp
@@
 	2100 6000 2150 6000
 Wire Wire Line
-	2150 6000 2150 5850
-Wire Wire Line
 	2100 6100 2250 6100
 Wire Wire Line
-	2100 6200 2450 6200
+	2100 6200 2300 6200
 Wire Wire Line
 	2450 6200 2450 6250
@@
 P 4400 3650
 F 0 "R1" V 4193 3650 50  0000 C CNN
-F 1 "R" V 4284 3650 50  0000 C CNN
+F 1 "1K" V 4284 3650 50  0000 C CNN
 F 2 "Resistor_SMD:R_0805_2012Metric_Pad1.15x1.40mm_HandSolder" V 4330 3650 50  0001 C CNN
 F 3 "~" H 4400 3650 50  0001 C CNN
@@
 P 5300 4050
 F 0 "R3" V 5093 4050 50  0000 C CNN
-F 1 "R" V 5184 4050 50  0000 C CNN
-F 2 "Resistor_SMD:R_0805_2012Metric_Pad1.15x1.40mm_HandSolder" V 5230 4050 50  0001 C CNN
+F 1 "3M" V 5184 4050 50  0000 C CNN
+F 2 "Resistor_THT:R_Axial_DIN0207_L6.3mm_D2.5mm_P2.54mm_Vertical" V 5230 4050 50  0001 C CNN
 F 3 "~" H 5300 4050 50  0001 C CNN
 	1    5300 4050
@@
 	5600 4300 5300 4300
 Wire Wire Line
-	4850 3650 4850 3850
-Wire Wire Line
 	4850 4200 4850 4300
 Wire Wire Line
 	5300 4300 4850 4300
 Connection ~ 5300 4300
-Wire Wire Line
-	5150 4050 5150 3850
-Wire Wire Line
-	5150 3850 4850 3850
-Connection ~ 4850 3850
-Wire Wire Line
-	4850 3850 4850 3900
 Wire Wire Line
 	5450 4050 5600 4050
@@
 P 4850 4050
 F 0 "C1" H 4965 4096 50  0000 L CNN
-F 1 "CP1" H 4965 4005 50  0000 L CNN
+F 1 "10µF" H 4965 4005 50  0000 L CNN
 F 2 "Capacitor_Tantalum_SMD:CP_EIA-3216-18_Kemet-A_Pad1.58x1.35mm_HandSolder" H 4850 4050 50  0001 C CNN
 F 3 "~" H 4850 4050 50  0001 C CNN
@@
 $EndComp
 Wire Wire Line
-	4950 3600 5800 3600
+	4950 3600 5150 3600
 Wire Wire Line
 	5600 3500 5600 4050
+Wire Wire Line
+	4850 3650 4850 3900
+Wire Wire Line
+	5150 3600 5150 4050
+Connection ~ 5150 3600
+Wire Wire Line
+	5150 3600 5800 3600
+$Comp
+L Device:CP1 C2
+U 1 1 5FE26281
+P 1550 6000
+F 0 "C2" H 1665 6046 50  0000 L CNN
+F 1 "100µF" H 1665 5955 50  0000 L CNN
+F 2 "Capacitor_THT:CP_Radial_D8.0mm_P3.80mm" H 1550 6000 50  0001 C CNN
+F 3 "~" H 1550 6000 50  0001 C CNN
+	1    1550 6000
+	-1   0    0    1
+$EndComp
+Wire Wire Line
+	2300 6200 2300 6400
+Wire Wire Line
+	2300 6400 1550 6400
+Wire Wire Line
+	1550 6400 1550 6150
+Connection ~ 2300 6200
+Wire Wire Line
+	2300 6200 2450 6200
+Wire Wire Line
+	2150 5600 2150 5700
+Wire Wire Line
+	1550 5850 1550 5700
+Wire Wire Line
+	1550 5700 2150 5700
+Connection ~ 2150 5700
+Wire Wire Line
+	2150 5700 2150 6000
 $EndSCHEMATC

Commit message: Board rework
Parts:
- removed C1: 10µF, Capacitor_Tantalum_SMD:CP_EIA-3216-18_Kemet-A_Pad1.58x1.35mm_HandSolder, symbol Device:CP1
- added Q2: 2N2219, Package_TO_SOT_THT:TO-92_Inline, symbol Transistor_BJT:2N2219
- C2: footprint Capacitor_THT:CP_Radial_D8.0mm_P3.80mm -> Capacitor_THT:CP_Radial_D8.0mm_P3.50mm
- R1: value 1K -> 470
- R3: value 3M -> 4.7K; footprint Resistor_THT:R_Axial_DIN0207_L6.3mm_D2.5mm_P2.54mm_Vertical -> Resistor_SMD:R_0805_2012Metric_Pad1.15x1.40mm_HandSolder
- renumbered J1 to 240VRelay1, J2 to 24V1, J6 to Fan1, J5 to Raspi1, J3 to Temp1, J4 to Temp2
Connections:
- net +5V: now also Temp1.1 (Pin_1), Temp2.1 (Pin_1); no longer R2.1, Temp1.3 (Pin_3), Temp2.3 (Pin_3)
- net GND: now also Temp1.3 (Pin_3), Temp2.3 (Pin_3), Q2.1 (E); no longer Temp1.1 (Pin_1), Temp2.1 (Pin_1)
- net TempData: now also R2.1; no longer R2.2
- net +3V3: now reaches Raspi1.1 (Pin_1)
- net +3V3: now also R2.2
- net at R1.1, R3.2: now also Q2.2 (B); no longer 240VRelay1.1 (Pin_1)
- new net: 240VRelay1.1 (Pin_1), Q2.3 (C)
Other:
- note added: "VCC\nData\nGND"
- note removed: "GND\nData\nVCC"
- moved on the sheet: 240VRelay1, C2, R1, R2, R3, Temp1, Temp2
